Commit message: Adding sensor plugins for imu camera and lidar and updating the leg joint limit values

File: src/urdf_and_meshes_of_the_robot/urdf/urdf_and_meshes_of_the_robot.urdf (robot description, URDF)
Before this commit: robot urdf_and_meshes_of_the_robot, 11 links, 10 joints
Joints:
- joint Left_joint: limit lower=0 upper=0 effort=0 velocity=0 -> lower=-1.57 upper=1.57 effort=5 velocity=1
- joint Lower_left_joint: limit lower=0 upper=0 effort=0 velocity=0 -> lower=-1.57 upper=1.57 effort=5 velocity=1
- joint Lower_right_joint: limit lower=0 upper=0 effort=0 velocity=0 -> lower=-1.57 upper=1.57 effort=5 velocity=1
- joint Upper_left_joint: limit lower=0 upper=0 effort=0 velocity=0 -> lower=-1.57 upper=1.57 effort=5 velocity=1
- joint Upper_right_joint: limit lower=0 upper=0 effort=0 velocity=0 -> lower=-1.57 upper=1.57 effort=5 velocity=1

Commit message: Updated on IMU sensor plugin and  Camera plugin

File: src/urdf_and_meshes_of_the_robot/urdf/urdf_and_meshes_of_the_robot.urdf (robot description, URDF)
Before this commit: robot urdf_and_meshes_of_the_robot, 11 links, 10 joints
Joints:
- removed joint Left_joint
- removed joint Right_joint
- added joint left_joint: type continuous, parent Lower_left_leg, child Left_wheel, origin xyz=0 -0.22885 0.015 rpy=3.1416 0 0.81783, axis 0 0 1, limit lower=-1.57 upper=1.57 effort=5 velocity=1
- added joint right_joint: type continuous, parent Lower_right_link, child Right_wheel, origin xyz=0 -0.22885 0.015 rpy=3.1416 0 0.41886, axis 0 0 1

Commit message: Updating RobotControlNode class in the robot_nodes_control.py script and introducing gazebo.launch.py file for rl training and refining all the sensors plugins to be error free.

File: src/urdf_and_meshes_of_the_robot/urdf/urdf_and_meshes_of_the_robot.urdf (robot description, URDF)
Before this commit: robot urdf_and_meshes_of_the_robot, 11 links, 10 joints
Links:
- added link camera_link_optical
Joints:
- removed joint left_joint
- removed joint right_joint
- added joint Left_joint: type continuous, parent Lower_left_leg, child Left_wheel, origin xyz=0 -0.22885 0.015 rpy=3.1416 0 0.81783, axis 0 0 1, limit lower=-1.57 upper=1.57 effort=5 velocity=1
- added joint Right_joint: type continuous, parent Lower_right_link, child Right_wheel, origin xyz=0 -0.22885 0.015 rpy=3.1416 0 0.41886, axis 0 0 1
- added joint camera_optical_joint: type fixed, parent camera_link, child camera_link_optical, origin xyz=0 0 0 rpy=-1.57079632679 0 -1.57079632679

Commit message: Fix camera orientation and add functional RL training with detailed progress tracking

File: src/urdf_and_meshes_of_the_robot/urdf/urdf_and_meshes_of_the_robot.urdf (robot description, URDF)
Before this commit: robot urdf_and_meshes_of_the_robot, 12 links, 11 joints
Links:
- link BODY_link: geometry collision mesh filename=package://urdf_and_meshes_of_the_robot/meshes/BODY_link.STL; visual mesh filename=package://urdf_and_meshes_of_the_robot/meshes/BODY_link.STL
- link IMU_link: geometry collision mesh filename=package://urdf_and_meshes_of_the_robot/meshes/IMU_link.STL; visual mesh filename=package://urdf_and_meshes_of_the_robot/meshes/IMU_link.STL
- link Left_wheel: geometry collision mesh filename=package://urdf_and_meshes_of_the_robot/meshes/Left_wheel.STL; visual mesh filename=package://urdf_and_meshes_of_the_robot/meshes/Left_wheel.STL
- link Lower_left_leg: geometry collision mesh filename=package://urdf_and_meshes_of_the_robot/meshes/Lower_left_le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; visual mesh filename=package://urdf_and_meshes_of_the_robot/meshes/Lower_left_le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
- link Lower_right_link: geometry collision mesh filename=package://urdf_and_meshes_of_the_robot/meshes/Lower_right_l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; visual mesh filename=package://urdf_and_meshes_of_the_robot/meshes/Lower_right_l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
- link Right_wheel: geometry collision mesh filename=package://urdf_and_meshes_of_the_robot/meshes/Right_wheel.S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; visual mesh filename=package://urdf_and_meshes_of_the_robot/meshes/Right_wheel.S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
- link Upper_left_leg: geometry collision mesh filename=package://urdf_and_meshes_of_the_robot/meshes/Upper_left_le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; visual mesh filename=package://urdf_and_meshes_of_the_robot/meshes/Upper_left_le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
- link Upper_right_link: geometry collision mesh filename=package://urdf_and_meshes_of_the_robot/meshes/Upper_right_l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; visual mesh filename=package://urdf_and_meshes_of_the_robot/meshes/Upper_right_l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
- link camera_link: geometry collision mesh filename=package://urdf_and_meshes_of_the_robot/meshes/camera_link.S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; visual mesh filename=package://urdf_and_meshes_of_the_robot/meshes/camera_link.S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
- link lidar_link: geometry collision mesh filename=package://urdf_and_meshes_of_the_robot/meshes/lidar_link.STL; visual mesh filename=package://urdf_and_meshes_of_the_robot/meshes/lidar_link.STL
Joints:
- joint camera_joint: origin xyz=0 -0.0868463319293926 0.00105377166734255 rpy=1.74532925199432 0 0 -> xyz=0 -0.0868463319293926 0.00105377166734255 rpy=1.57 0 -1.57
