Commit message: MuJoCo migration: from-scratch PPO balances on wheels, yaw-stable
Move balance training to MuJoCo, where the load-bearing revolute leg joints
actually hold under load (Gazebo Classic could not), so the robot is a real
inverted pendulum on its wheels and the hand-written PPO gets a genuine
balance signal.

- mujoco/mybot.xml: floating-base model (2 wheel torque actuators, 8 leg PD
  position servos, IMU sensors, external tracking camera, 1280x720 offscreen)
- balance_env_mujoco.py: Gymnasium env, 69-d proprioceptive obs (3-frame
  history), 2 wheel-torque action, reward = alive - tilt^2 - drift^2 - yaw^2
  - action^2; terminates on fall
- ppo_balance.py: --env mujoco path; decoupled save scheme (best/latest/every-N
  episodes); target-kl + ent-coef stabilization (KL cap prevents policy blowup)
- mujoco_record.py (headless osmesa mp4), mujoco_play.py (live viewer),
  yaw_compare.py (before/after rollout metrics)
- Yaw-rate penalty stops in-place spinning: mean yaw-rate 230 -> 18 deg/s,
  heading held to ~4 deg, still balances the full 1000-step episode
- README rewrite (MuJoCo primary path) + CLAUDE.md working guide
- Gazebo Classic + ros2_control path kept as legacy/reference

File: src/urdf_and_meshes_of_the_robot/urdf/mybot_balance.urdf.xacro (robot description, xacro)
@@ -91,45 +91,74 @@
       <state_interface name="effort"/>
     </joint>
-    <!-- ===== Legs: position control (held at zero stance for balance) ===== -->
+    <!-- ===== Legs: ONLY ros2_control-managed when NOT locked (revolute walking stage).
+         With lock_legs=true the leg joints are FIXED (rigid balance stance) and must not
+         appear here — a fixed joint has no command interface. position_pid + gains are
+         kept for the future walking stage (set lock_legs:=false + spawn the controller). -->
+    <xacro:unless value="$(arg lock_legs)">
     <joint name="hip_yaw_left">
-      <command_interface name="position"/>
+      <command_interface name="effort">
+        <param name="min">-200.0</param>
+        <param name="max">200.0</param>
+      </command_interface>
       <state_interface name="position"/>
       <state_interface name="velocity"/>
     </joint>
     <joint name="hip_roll_left">
-      <command_interface name="position"/>
+      <command_interface name="effort">
+        <param name="min">-200.0</param>
+        <param name="max">200.0</param>
+      </command_interface>
       <state_interface name="position"/>
       <state_interface name="velocity"/>
     </joint>
     <joint name="Upper_left_joint">
-      <command_interface name="position"/>
+      <command_interface name="effort">
+        <param name="min">-200.0</param>
+        <param name="max">200.0</param>
+      </command_interface>
       <state_interface name="position"/>
       <state_interface name="velocity"/>
     </joint>
     <joint name="Lower_left_joint">
-      <command_interface name="position"/>
+      <command_interface name="effort">
+        <param name="min">-200.0</param>
+        <param name="max">200.0</param>
+      </command_interface>
       <state_interface name="position"/>
       <state_interface name="velocity"/>
     </joint>
     <joint name="hip_yaw_right">
-      <command_interface name="position"/>
+      <command_interface name="effort">
+        <param name="min">-200.0</param>
+        <param name="max">200.0</param>
+      </command_interface>
       <state_interface name="position"/>
       <state_interface name="velocity"/>
     </joint>
     <joint name="hip_roll_right">
-      <command_interface name="position"/>
+      <command_interface name="effort">
+        <param name="min">-200.0</param>
+        <param name="max">200.0</param>
+      </command_interface>
       <state_interface name="position"/>
       <state_interface name="velocity"/>
     </joint>
     <joint name="Upper_right_joint">
-      <command_interface name="position"/>
+      <command_interface name="effort">
+        <param name="min">-200.0</param>
+        <param name="max">200.0</param>
+      </command_interface>
       <state_interface name="position"/>
       <state_interface name="velocity"/>
     </joint>
     <joint name="Lower_right_joint">
-      <command_interface name="position"/>
+      <command_interface name="effort">
+        <param name="min">-200.0</param>
+        <param name="max">200.0</param>
+      </command_interface>
       <state_interface name="position"/>
       <state_interface name="velocity"/>
     </joint>
+    </xacro:unless>
   </ros2_control>
   <!-- ============================================================= -->

File: src/urdf_and_meshes_of_the_robot/urdf/mybot_geometry.urdf.xacro (robot description, xacro)
@@ -1,4 +1,12 @@
 <?xml version="1.0"?>
 <robot name="urdf_and_meshes_of_the_robot" xmlns:xacro = "http://ros.org/wiki/xacro">
+  <!-- lock_legs: 'true' => the 8 leg joints are FIXED (rigid inverted-pendulum stance
+       for the STAGE-1 balance task; the wheels alone must keep the tall body upright).
+       'false' => the legs are 'revolute' + position_pid (for a later walking stage).
+       gazebo_ros2_control cannot hold these load-bearing chained joints via a position
+       interface (they buckle + kinematically lock), so we fix them for balance.
+       The balance launch passes this via xacro mappings; default = fixed. -->
+  <xacro:arg name="lock_legs" default="true"/>
+  <xacro:property name="_ljt" value="${'fixed' if '$(arg lock_legs)' == 'true' else 'revolute'}"/>
   <link name="base_link"/>  <!-- Dummy link added -->
   <joint name="base_joint" type="fixed">
@@ -92,11 +100,11 @@
        cylinders (no STL needed). NOTE: yaw axis = Z (vertical), roll axis = X (forward);
        verify/flip in RViz if the sense looks wrong for your build. -->
-  <joint name="hip_yaw_left" type="revolute">   <!-- free leg joint: actuated, held at stance for balance; RL-controlled for walking -->
+  <joint name="hip_yaw_left" type="${_ljt}">   <!-- free leg joint: actuated, held at stance for balance; RL-controlled for walking -->
     <origin xyz="0.065 -0.0025 -0.055" rpy="0 0 0" />
     <parent link="BODY_link" />
     <child link="hip_yaw_link_left" />
     <axis xyz="0 0 1" />
-    <limit lower="-0.785" upper="0.785" effort="20" velocity="10" />
-    <dynamics damping="10.0" friction="100.0"/>
+    <limit lower="-0.785" upper="0.785" effort="200" velocity="10" />
+    <dynamics damping="0.5" friction="0.1"/>
   </joint>
   <link name="hip_yaw_link_left">
@@ -113,11 +121,11 @@
     </visual>
   </link>
-  <joint name="hip_roll_left" type="revolute">   <!-- free leg joint: actuated, held at stance for balance; RL-controlled for walking -->
+  <joint name="hip_roll_left" type="${_ljt}">   <!-- free leg joint: actuated, held at stance for balance; RL-controlled for walking -->
     <origin xyz="0 0 0" rpy="0 0 0" />
     <parent link="hip_yaw_link_left" />
     <child link="hip_roll_link_left" />
     <axis xyz="1 0 0" />
-    <limit lower="-0.785" upper="0.785" effort="20" velocity="10" />
-    <dynamics damping="10.0" friction="100.0"/>
+    <limit lower="-0.785" upper="0.785" effort="200" velocity="10" />
+    <dynamics damping="0.5" friction="0.1"/>
   </joint>
   <link name="hip_roll_link_left">
@@ -136,5 +144,5 @@
   <joint
     name="Upper_left_joint"
-    type="revolute">   <!-- free leg joint: actuated, held at stance for balance; RL-controlled for walking -->
+    type="${_ljt}">   <!-- free leg joint: actuated, held at stance for balance; RL-controlled for walking -->
     <origin
       xyz="0 0 0"
@@ -149,7 +157,7 @@
       lower="-1.57"
       upper="1.57"
-      effort="20"
+      effort="200"
       velocity="30" />
-    <dynamics damping="10.0" friction="100.0"/>
+    <dynamics damping="0.5" friction="0.1"/>
   </joint>
   <link
@@ -195,5 +203,5 @@
   <joint
     name="Lower_left_joint"
-    type="revolute">   <!-- free leg joint: actuated, held at stance for balance; RL-controlled for walking -->
+    type="${_ljt}">   <!-- free leg joint: actuated, held at stance for balance; RL-controlled for walking -->
     <origin
       xyz="0 -0.24941 0.032"
@@ -208,7 +216,7 @@
       lower="-1.57"
       upper="1.57"
-      effort="20"
+      effort="200"
       velocity="30" />
-    <dynamics damping="10.0" friction="100.0"/>
+    <dynamics damping="0.5" friction="0.1"/>
   </joint>
   <link
@@ -265,5 +273,5 @@
       lower="-1.57"
       upper="1.57"
-      effort="20"
+      effort="200"
       velocity="30" />
   </joint>
@@ -309,11 +317,11 @@
   </link>
   <!-- ===================== RIGHT HIP : 3-DOF (yaw -> roll -> pitch) ===================== -->
-  <joint name="hip_yaw_right" type="revolute">   <!-- free leg joint: actuated, held at stance for balance; RL-controlled for walking -->
+  <joint name="hip_yaw_right" type="${_ljt}">   <!-- free leg joint: actuated, held at stance for balance; RL-controlled for walking -->
     <origin xyz="-0.065 -0.0025 -0.055" rpy="0 0 0" />
     <parent link="BODY_link" />
     <child link="hip_yaw_link_right" />
     <axis xyz="0 0 1" />
-    <limit lower="-0.785" upper="0.785" effort="20" velocity="10" />
-    <dynamics damping="10.0" friction="100.0"/>
+    <limit lower="-0.785" upper="0.785" effort="200" velocity="10" />
+    <dynamics damping="0.5" friction="0.1"/>
   </joint>
   <link name="hip_yaw_link_right">
@@ -330,11 +338,11 @@
     </visual>
   </link>
-  <joint name="hip_roll_right" type="revolute">   <!-- free leg joint: actuated, held at stance for balance; RL-controlled for walking -->
+  <joint name="hip_roll_right" type="${_ljt}">   <!-- free leg joint: actuated, held at stance for balance; RL-controlled for walking -->
     <origin xyz="0 0 0" rpy="0 0 0" />
     <parent link="hip_yaw_link_right" />
     <child link="hip_roll_link_right" />
     <axis xyz="1 0 0" />
-    <limit lower="-0.785" upper="0.785" effort="20" velocity="10" />
-    <dynamics damping="10.0" friction="100.0"/>
+    <limit lower="-0.785" upper="0.785" effort="200" velocity="10" />
+    <dynamics damping="0.5" friction="0.1"/>
   </joint>
   <link name="hip_roll_link_right">
@@ -353,5 +361,5 @@
   <joint
     name="Upper_right_joint"
-    type="revolute">   <!-- free leg joint: actuated, held at stance for balance; RL-controlled for walking -->
+    type="${_ljt}">   <!-- free leg joint: actuated, held at stance for balance; RL-controlled for walking -->
     <origin
       xyz="0 0 0"
@@ -366,7 +374,7 @@
       lower="-1.57"
       upper="1.57"
-      effort="20"
+      effort="200"
       velocity="30" />
-    <dynamics damping="10.0" friction="100.0"/>
+    <dynamics damping="0.5" friction="0.1"/>
   </joint>
   <link
@@ -412,5 +420,5 @@
   <joint
     name="Lower_right_joint"
-    type="revolute">   <!-- free leg joint: actuated, held at stance for balance; RL-controlled for walking -->
+    type="${_ljt}">   <!-- free leg joint: actuated, held at stance for balance; RL-controlled for walking -->
     <origin
       xyz="0 -0.24941 0.034"
@@ -425,7 +433,7 @@
       lower="-1.57"
       upper="1.57"
-      effort="20"
+      effort="200"
       velocity="30" />
-    <dynamics damping="10.0" friction="100.0"/>
+    <dynamics damping="0.5" friction="0.1"/>
   </joint>
   <link
